File: hardware/RetroLink.brd (EAGLE design)
At the start: 35.2 x 20.3 mm, 16 parts, among them J2 MICROXNJ, SW1 SKRPABE010, U1 CH559L, U2 CH340N, U3 LM66100DCKR, X1 PN87520-S, X3 DB9

Commit message: hardware changes
Parts:
- R1: value 470 -> 330
Other:
- board text added: "Config"
- board text added: "RetroLink"
- board text added: "v1.4"
- board text removed: "DB9"
- board text removed: "v1.3"
Changed lines of the file:
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@@
 <wire x1="35.23" y1="22.85" x2="0" y2="22.85" width="0" layer="20"/>
 <wire x1="0" y1="22.85" x2="0" y2="2.54" width="0" layer="20"/>
-<text x="31.369" y="10.922" size="1.27" layer="25" rot="R90">DB9</text>
-<text x="0.635" y="3.175" size="1.016" layer="25">https://github.com/fbeen/retrolink</text>
-<text x="32.004" y="3.175" size="1.016" layer="25">v1.3</text>
+<text x="25.908" y="17.272" size="1.016" layer="25">Config</text>
+<text x="0.381" y="3.048" size="0.8128" layer="25">https://github.com/fbeen/retrolink</text>
+<text x="32.004" y="3.175" size="1.016" layer="25">v1.4</text>
+<text x="1.651" y="21.336" size="1.016" layer="25">RetroLink</text>
 </plain>
 <attributes>
@@
 <elements>
 <element name="C6" library="rcl" library_urn="urn:adsk.eagle:library:334" package="C0603" package3d_urn="urn:adsk.eagle:package:23616/2" value="100nf" x="10.922" y="6.858" smashed="yes" rot="R90">
-<attribute name="NAME" x="10.287" y="5.715" size="1.27" layer="25" rot="R90"/>
+<attribute name="NAME" x="10.287" y="5.715" size="1.016" layer="25" rot="R90"/>
 <attribute name="POPULARITY" value="73" x="51.562" y="43.688" size="1.778" layer="27" rot="R90" display="off"/>
 <attribute name="SPICEPREFIX" value="C" x="51.562" y="43.688" size="1.778" layer="27" rot="R90" display="off"/>
@@
 </element>
 <element name="C3" library="rcl" library_urn="urn:adsk.eagle:library:334" package="C0603" package3d_urn="urn:adsk.eagle:package:23616/2" value="4.7Uf" x="17.907" y="7.366" smashed="yes">
-<attribute name="NAME" x="16.764" y="8.001" size="1.27" layer="25"/>
+<attribute name="NAME" x="16.764" y="8.001" size="1.016" layer="25"/>
 <attribute name="POPULARITY" value="73" x="67.437" y="-33.274" size="1.778" layer="27" display="off"/>
 <attribute name="SPICEPREFIX" value="C" x="67.437" y="-33.274" size="1.778" layer="27" display="off"/>
 </element>
 <element name="C4" library="rcl" library_urn="urn:adsk.eagle:library:334" package="C0603" package3d_urn="urn:adsk.eagle:package:23616/2" value="10Uf" x="22.479" y="17.78" smashed="yes">
-<attribute name="NAME" x="18.923" y="16.764" size="1.27" layer="25"/>
+<attribute name="NAME" x="18.923" y="16.764" size="1.016" layer="25"/>
 <attribute name="POPULARITY" value="73" x="40.259" y="-30.48" size="1.778" layer="27" display="off"/>
 <attribute name="SPICEPREFIX" value="C" x="40.259" y="-30.48" size="1.778" layer="27" display="off"/>
@@
 </element>
 <element name="U1" library="CH559L" package="TQFP48_7X7" value="CH559L" x="24.765" y="8.255" smashed="yes" rot="R90">
-<attribute name="NAME" x="31.877" y="5.969" size="1.27" layer="25" rot="R180"/>
+<attribute name="NAME" x="29.845" y="12.7" size="1.016" layer="25" rot="R180"/>
 </element>
 <element name="X3" library="con-subd" library_urn="urn:adsk.eagle:library:189" package="F09D" package3d_urn="urn:adsk.eagle:package:10273/1" value="DB9" x="39.37" y="12.7" smashed="yes" rot="R270">
@@
 <attribute name="MF" value="WCH" x="12.7" y="12.7" size="1.778" layer="27" rot="R270" display="off"/>
 <attribute name="MP" value="CH340N" x="12.7" y="12.7" size="1.778" layer="27" rot="R270" display="off"/>
-<attribute name="NAME" x="10.033" y="11.557" size="1.27" layer="25" rot="R90"/>
+<attribute name="NAME" x="10.033" y="11.557" size="1.016" layer="25" rot="R90"/>
 <attribute name="PACKAGE" value="Package " x="12.7" y="12.7" size="1.778" layer="27" rot="R270" display="off"/>
 <attribute name="PRICE" value="None" x="12.7" y="12.7" size="1.778" layer="27" rot="R270" display="off"/>
@@
 </element>
 <element name="C1" library="rcl" library_urn="urn:adsk.eagle:library:334" package="C0603" package3d_urn="urn:adsk.eagle:package:23616/2" value="100nf" x="17.907" y="9.779" smashed="yes">
-<attribute name="NAME" x="16.764" y="10.414" size="1.27" layer="25"/>
+<attribute name="NAME" x="16.764" y="10.414" size="1.016" layer="25"/>
 <attribute name="POPULARITY" value="73" x="17.907" y="9.779" size="1.778" layer="27" display="off"/>
 <attribute name="SPICEPREFIX" value="C" x="17.907" y="9.779" size="1.778" layer="27" display="off"/>
@@
 </element>
 <element name="LED1" library="led" library_urn="urn:adsk.eagle:library:259" package="SML0603" package3d_urn="urn:adsk.eagle:package:15832/1" value="Status" x="17.526" y="15.367" smashed="yes">
-<attribute name="NAME" x="15.621" y="13.462" size="1.27" layer="25"/>
+<attribute name="NAME" x="15.621" y="13.462" size="1.016" layer="25"/>
 <attribute name="POPULARITY" value="17" x="17.526" y="15.367" size="1.778" layer="27" display="off"/>
 <attribute name="VALUE" x="16.526" y="13.367" size="1.27" layer="27"/>
 </element>
-<element name="R1" library="rcl" library_urn="urn:adsk.eagle:library:334" package="R0603" package3d_urn="urn:adsk.eagle:package:23555/3" value="470" x="20.955" y="15.367" smashed="yes">
-<attribute name="NAME" x="20.32" y="13.462" size="1.27" layer="25"/>
+<element name="R1" library="rcl" library_urn="urn:adsk.eagle:library:334" package="R0603" package3d_urn="urn:adsk.eagle:package:23555/3" value="330" x="20.955" y="15.367" smashed="yes">
+<attribute name="NAME" x="20.32" y="13.462" size="1.016" layer="25"/>
 <attribute name="POPULARITY" value="70" x="20.955" y="15.367" size="1.778" layer="27" display="off"/>
 <attribute name="SPICEPREFIX" value="R" x="20.955" y="15.367" size="1.778" layer="27" display="off"/>
@@
 <attribute name="MF" value="Shouhan" x="14.605" y="22.86" size="1.778" layer="27" display="off"/>
 <attribute name="MP" value="MICROXNJ" x="14.605" y="22.86" size="1.778" layer="27" display="off"/>
-<attribute name="NAME" x="10.405" y="16.76" size="1.27" layer="25" align="top-left"/>
 <attribute name="PACKAGE" value="Package " x="14.605" y="22.86" size="1.778" layer="27" display="off"/>
 <attribute name="PRICE" value="None" x="14.605" y="22.86" size="1.778" layer="27" display="off"/>
