File: hardware/RetroLink.sch (EAGLE design)
At the start: 16 parts, among them J2 MICROXNJ, SW1 SKRPABE010, U1 CH559L, U2 CH340N, U3 LM66100DCKR, X1 PN87520-S, X3 DB9

Commit message: hardware changes
Parts:
- R1: value 470 -> 330
Changed lines of the file:
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@@
 <part name="GND13" library="supply1" library_urn="urn:adsk.eagle:library:371" deviceset="GND" device=""/>
 <part name="LED1" library="led" library_urn="urn:adsk.eagle:library:259" deviceset="LED" device="SML0603" package3d_urn="urn:adsk.eagle:package:15832/1" value="Status"/>
-<part name="R1" library="rcl" library_urn="urn:adsk.eagle:library:334" deviceset="R-EU_" device="R0603" package3d_urn="urn:adsk.eagle:package:23555/3" value="470"/>
+<part name="R1" library="rcl" library_urn="urn:adsk.eagle:library:334" deviceset="R-EU_" device="R0603" package3d_urn="urn:adsk.eagle:package:23555/3" value="330"/>
 <part name="GND14" library="supply1" library_urn="urn:adsk.eagle:library:371" deviceset="GND" device=""/>
 <part name="X1" library="con-berg" library_urn="urn:adsk.eagle:library:130" deviceset="PN87520-S" device="" package3d_urn="urn:adsk.eagle:package:6147/1"/>
